Commit message: update the description file

File: iaac_ur_description/urdf/deco2_mosaic.xacro (robot description, xacro)
@@ -8,26 +8,34 @@
   <!-- Include base robot definition -->
   <xacro:include filename="$(find ur_description)/urdf/ur.urdf.xacro"/>
+  <link name="tcp_ee"/>
+  <joint name="deco2_ee" type="fixed">
+    <parent link="tool0"/>
+    <child link="tcp_ee"/>
+    <origin xyz="0.0015 0.00255 0.13502" rpy="0 0 0"/> <!-- TCP location -->
+  </joint>
   <!-- Add end-effector frame -->
   <link name="suction_cup_frame">
     <visual>
-      <origin xyz="0 0 0" rpy="0 0 0"/>
+      <origin xyz="0 0 0" rpy="0 0 -1.5708"/>
       <geometry>
-        <box size="0.02 0.02 0.02"/> <!-- Placeholder visual -->
+        <!-- <box size="0.02 0.02 0.02"/>  -->
+        <mesh filename="package://iaac_ur_description/meshes/deco2/deco2_ee_vi.stl" scale="1 1 1"/>
       </geometry>
       <material name="placeholder_grey">
-        <color rgba="0.6 0.6 0.6 1.0"/>
+        <color rgba="0.851 0.439 0.106 0.8"/>
       </material>
     </visual>
     <collision>
-      <origin xyz="0 0 0" rpy="0 0 0"/>
+      <origin xyz="0 0 0" rpy="0 0 -1.5708"/>
       <geometry>
-        <box size="0.02 0.02 0.02"/> <!-- Placeholder collision -->
+        <!-- <box size="0.02 0.02 0.02"/>  -->
+        <mesh filename="package://iaac_ur_description/meshes/deco2/deco2_ee_co.stl" scale="1 1 1"/>
       </geometry>
     </collision>
   </link>
   <joint name="vaccum_gripper" type="fixed">
-    <parent link="tool0"/>  <!-- replace with correct parent link if needed -->
+    <parent link="tcp_ee"/> <!-- Attach to the end-effector -->
     <child link="suction_cup_frame"/>
-    <origin xyz="0 0 0.0" rpy="0 0 0"/> <!-- adjust this to position the EE correctly -->
+    <origin xyz="-0.0015 -0.00255 -0.13502" rpy="0 0 0"/> <!-- adjust this to position the EE correctly -->
   </joint>
 </robot>

Commit message: update notebook

File: iaac_ur_description/urdf/deco2_mosaic.xacro (robot description, xacro)
@@ -39,3 +39,9 @@
     <origin xyz="-0.0015 -0.00255 -0.13502" rpy="0 0 0"/> <!-- adjust this to position the EE correctly -->
   </joint>
+  <link name="camera_color_optical_frame"/>
+  <joint name="camera_link" type="fixed">
+    <parent link="tool0"/>  <!-- or "tcp_ee" if camera is mounted on EE -->
+    <child link="camera_color_optical_frame"/>
+    <origin xyz="0.074355 -0.103473 -0.020089" rpy="-0.0040865 0.0067126 -0.0100596"/>
+  </joint>
 </robot>

Commit message: update calibration data

File: iaac_ur_description/urdf/deco2_mosaic.xacro (robot description, xacro)
@@ -37,5 +37,5 @@
     <parent link="tcp_ee"/> <!-- Attach to the end-effector -->
     <child link="suction_cup_frame"/>
-    <origin xyz="-0.0015 -0.00255 -0.13502" rpy="0 0 0"/> <!-- adjust this to position the EE correctly -->
+    <origin xyz="-0.00312 -0.00017 -0.13501" rpy="0 0 0"/> <!-- adjust this to position the EE correctly -->
   </joint>
   <link name="camera_color_optical_frame"/>
@@ -43,5 +43,5 @@
     <parent link="tool0"/>  <!-- or "tcp_ee" if camera is mounted on EE -->
     <child link="camera_color_optical_frame"/>
-    <origin xyz="0.074355 -0.103473 -0.020089" rpy="-0.0040865 0.0067126 -0.0100596"/>
+    <origin xyz="0.083810 -0.108334 -0.029525" rpy="-0.011312 0.0000671 -0.0016056"/>
   </joint>
 </robot>

Commit message: add handeye for the workshop

File: iaac_ur_description/urdf/deco2_mosaic.xacro (robot description, xacro)
@@ -12,5 +12,5 @@
     <parent link="tool0"/>
     <child link="tcp_ee"/>
-    <origin xyz="0.0015 0.00255 0.13502" rpy="0 0 0"/> <!-- TCP location -->
+    <origin xyz="0.00312 0.00186 0.13315" rpy="0 0 0"/> <!-- TCP location -->
   </joint>
   <!-- Add end-effector frame -->
@@ -37,5 +37,5 @@
     <parent link="tcp_ee"/> <!-- Attach to the end-effector -->
     <child link="suction_cup_frame"/>
-    <origin xyz="-0.00312 -0.00017 -0.13501" rpy="0 0 0"/> <!-- adjust this to position the EE correctly -->
+    <origin xyz="-0.00312 -0.00186 -0.13315" rpy="0 0 0"/> <!-- adjust this to position the EE correctly -->
   </joint>
   <link name="camera_color_optical_frame"/>
@@ -43,5 +43,5 @@
     <parent link="tool0"/>  <!-- or "tcp_ee" if camera is mounted on EE -->
     <child link="camera_color_optical_frame"/>
-    <origin xyz="0.083810 -0.108334 -0.029525" rpy="-0.011312 0.0000671 -0.0016056"/>
+    <origin xyz="0.087143 -0.104806 0.030877" rpy="-0.0058639 0.0005677 -0.0074144"/>
   </joint>
 </robot>
